Commit message: debugging

File: ros_ws/install/scout_mini_description/share/scout_mini_description/urdf/scout_mini.urdf.xacro (robot description, xacro)
@@ -1,174 +1 @@
-<?xml version="1.0"?>
-<robot xmlns:xacro="http://www.ros.org/wiki/xacro" name="scout_mini">
-  <xacro:property name="PI" value="3.1415926535897931" />
-  <link name="base_link">
-    <visual>
-      <origin xyz="0 0 0.0" rpy="${PI/2} 0 -${PI/2}" />
-      <geometry>
-        <mesh filename="package://scout_mini_description/meshes/body.dae" />
-      </geometry>
-    </visual>
-    <collision>
-      <origin xyz="0 0 0" rpy="0 0 0" />
-      <geometry>
-        <box size="0.514618 0.3816 0.10357" />
-      </geometry>
-    </collision>
-  </link>
-  <joint name="inertial_joint" type="fixed">
-    <parent link="base_link" />
-    <child link="inertial_link" />
-    <origin xyz="0 0 0" rpy="0 0 0" />
-  </joint>
-  <link name="inertial_link">
-    <inertial>
-      <mass value="60" />
-      <origin xyz="0 0 0" rpy="0 0 0" />
-      <inertia ixx="2.288641" ixy="0" ixz="0" iyy="5.103976" iyz="0" izz="3.431465" />
-    </inertial>
-  </link>
-  <joint name="front_left_wheel_joint" type="continuous">
-    <parent link="base_link" />
-    <child link="front_left_wheel_link" />
-    <origin xyz="0.2319755 0.245 -0.100998" rpy="0 0 0" />
-    <axis xyz="0 1 0" rpy="0 0 0" />
-  </joint>
-  <link name="front_left_wheel_link">
-    <visual>
-      <origin xyz="0 -0.0367485 0" rpy="-${PI/2} 0 0" />
-      <geometry>
-        <mesh filename="package://scout_mini_description/meshes/wheel.dae" />
-      </geometry>
-    </visual>
-    <collision>
-      <origin xyz="0 -0.0367485 0" rpy="-${PI/2} 0 0" />
-      <geometry>
-        <mesh filename="package://scout_mini_description/meshes/wheel.dae" />
-      </geometry>
-    </collision>
-    <inertial>
-      <mass value="15" />
-      <origin xyz="0 0 0" rpy="0 0 0" />
-      <inertia ixx="0.6171" ixy="0" ixz="0" iyy="0.6171" iyz="0" izz="0.1361" />
-    </inertial>
-  </link>
-  <joint name="rear_left_wheel_joint" type="continuous">
-    <parent link="base_link" />
-    <child link="rear_left_wheel_link" />
-    <origin xyz="-0.2319755 0.245 -0.100998" rpy="0 0 0" />
-    <axis xyz="0 1 0" rpy="0 0 0" />
-  </joint>
-  <link name="rear_left_wheel_link">
-    <visual>
-      <origin xyz="0 -0.0367485 0" rpy="-${PI/2} 0 0" />
-      <geometry>
-        <mesh filename="package://scout_mini_description/meshes/wheel.dae" />
-      </geometry>
-    </visual>
-    <collision>
-      <origin xyz="0 -0.0367485 0" rpy="-${PI/2} 0 0" />
-      <geometry>
-        <mesh filename="package://scout_mini_description/meshes/wheel.dae" />
-      </geometry>
-    </collision>
-    <inertial>
-      <mass value="15" />
-      <origin xyz="0 0 0" rpy="0 0 0" />
-      <inertia ixx="0.6171" ixy="0" ixz="0" iyy="0.6171" iyz="0" izz="0.1361" />
-    </inertial>
-  </link>
-  <joint name="front_right_wheel_joint" type="continuous">
-    <parent link="base_link" />
-    <child link="front_right_wheel_link" />
-    <origin xyz="0.2319755 -0.245 -0.099998" rpy="0 0 0" />
-    <axis xyz="0 1 0" rpy="0 0 0" />
-  </joint>
-  <link name="front_right_wheel_link">
-    <visual>
-      <origin xyz="0 0.0367485 0" rpy="${PI/2} 0 0" />
-      <geometry>
-        <mesh filename="package://scout_mini_description/meshes/wheel.dae" />
-      </geometry>
-    </visual>
-    <collision>
-      <origin xyz="0 0.0367485 0" rpy="${PI/2} 0 0" />
-      <geometry>
-        <mesh filename="package://scout_mini_description/meshes/wheel.dae" />
-      </geometry>
-    </collision>
-    <inertial>
-      <mass value="15" />
-      <origin xyz="0 0 0" rpy="0 0 0" />
-      <inertia ixx="0.6171" ixy="0" ixz="0" iyy="0.6171" iyz="0" izz="0.1361" />
-    </inertial>
-  </link>
-  <joint name="rear_right_wheel_joint" type="continuous">
-    <parent link="base_link" />
-    <child link="rear_right_wheel_link" />
-    <origin xyz="-0.2319755 -0.245 -0.099998" rpy="0 0 0" />
-    <axis xyz="0 1 0" rpy="0 0 0" />
-  </joint>
-  <link name="rear_right_wheel_link">
-    <visual>
-      <origin xyz="0 0.0367485 0" rpy="${PI/2} 0 0" />
-      <geometry>
-        <mesh filename="package://scout_mini_description/meshes/wheel.dae" />
-      </geometry>
-    </visual>
-    <collision>
-      <origin xyz="0 0.0367485 0" rpy="${PI/2} 0 0" />
-      <geometry>
-        <mesh filename="package://scout_mini_description/meshes/wheel.dae" />
-      </geometry>
-    </collision>
-    <inertial>
-      <mass value="15" />
-      <origin xyz="0 0 0" rpy="0 0 0" />
-      <inertia ixx="0.6171" ixy="0" ixz="0" iyy="0.6171" iyz="0" izz="0.1361" />
-    </inertial>
-  </link>
-  <ros2_control name="scout_mini_control" type="system">
-    <hardware>
-      <plugin>scout_mini_hardware/ScoutMiniHardware</plugin>
-      <param name="interface">can0</param>
-      <param name="wheel_radius">0.0875</param>
-      <param name="wheel_separation">0.490</param>
-    </hardware>
-    <joint name="front_left_wheel_joint">
-      <command_interface name="velocity">
-        <param name="min">-1</param>
-        <param name="max">1</param>
-      </command_interface>
-      <state_interface name="position" />
-      <state_interface name="velocity" />
-      <state_interface name="effort" />
-    </joint>
-    <joint name="rear_left_wheel_joint">
-      <command_interface name="velocity">
-        <param name="min">-1</param>
-        <param name="max">1</param>
-      </command_interface>
-      <state_interface name="position" />
-      <state_interface name="velocity" />
-      <state_interface name="effort" />
-    </joint>
-    <joint name="front_right_wheel_joint">
-      <command_interface name="velocity">
-        <param name="min">-1</param>
-        <param name="max">1</param>
-      </command_interface>
-      <state_interface name="position" />
-      <state_interface name="velocity" />
-      <state_interface name="effort" />
-    </joint>
-    <joint name="rear_right_wheel_joint">
-      <command_interface name="velocity">
-        <param name="min">-1</param>
-        <param name="max">1</param>
-      </command_interface>
-      <state_interface name="position" />
-      <state_interface name="velocity" />
-      <state_interface name="effort" />
-    </joint>
-  </ros2_control>
-</robot>
+/apollo/ros_ws/src/scout_mini_description/urdf/scout_mini.urdf.xacro
